Commit message: initial full simulation implementation and documentation

File: dependencies/catamaran/urdf/catamaran.urdf (robot description, URDF)
Before this commit: robot catamaran, 5 links, 4 joints
Links:
- link l_thruster: mass 0 -> 5
- link mount: mass 0 -> 10
- link r_thruster: mass 0 -> 5

Commit message: fixed simulation

File: dependencies/catamaran/urdf/catamaran.urdf (robot description, URDF)
Before this commit: robot catamaran, 5 links, 4 joints
Links:
- link base_link: mass 60.344 -> 100
- link l_thruster: mass 5 -> 80
- link mount: mass 10 -> 17.43
- link r_thruster: mass 5 -> 80
Joints:
- removed joint base_to_l_thruster
- added joint base_to_l_thrruster: type fixed, parent base_link, child l_thruster, origin xyz=0.55834 0.43963 -0.45538 rpy=1.5708 0 3.1416, axis 0 0 0
- joint base_to_mount: origin xyz=0 -0.060366 0.14462 rpy=1.5708 0 0 -> xyz=0 -0.31037 0.14462 rpy=1.5708 0 0

Commit message: fixed simulation, added velocity control

File: dependencies/catamaran/urdf/catamaran.urdf (robot description, URDF)
Before this commit: robot catamaran, 5 links, 4 joints
Links:
- link base_link: mass 100 -> 60.33169
- link l_thruster: mass 80 -> None; geometry visual mesh filename=package://catamaran/meshes/l_thruster.STL
- link r_thruster: mass 80 -> None; geometry visual mesh filename=package://catamaran/meshes/r_thruster.STL

File: triton/urdf/catamaran_full.urdf.xacro (robot description, xacro)
@@ -23,4 +23,8 @@
           </right_force_point>
         </plugin>
+        <plugin name="VelocityPlugin" filename="libvelocity_plugin.so">
+          <link_name>base_footprint</link_name>
+          <ros_topic>velocity</ros_topic>
+        </plugin>
     </gazebo>
 </robot>

Commit message: added competition simulation

File: dependencies/catamaran/urdf/catamaran.urdf (robot description, URDF)
Before this commit: robot catamaran, 5 links, 4 joints
Links:
- removed link mount
- added link waterwheel, mass 11.524; visual mesh filename=package://catamaran/meshes/waterwheel.STL
- link base_link: mass 60.33169 -> 682.95
- link l_thruster: mass None -> 4.9984
- link r_thruster: mass None -> 0
Joints:
- removed joint base_to_l_thrruster
- removed joint base_to_mount
- added joint base_to_l_thruster: type fixed, parent base_link, child l_thruster, origin xyz=0.55834 0.43963 -0.45538 rpy=1.5708 0 3.1416, axis 0 0 0
- added joint base_to_waterwheel: type fixed, parent base_link, child waterwheel, origin xyz=0 -0.68537 -0.15538 rpy=1.5708 0 0, axis 1 0 0

File: triton/urdf/catamaran_full.urdf.xacro (robot description, xacro)
@@ -6,9 +6,9 @@
     <xacro:include filename="$(find velodyne_description)/urdf/VLP-16.urdf.xacro"/>
     <xacro:include filename="$(find realsense_ros_gazebo)/xacro/depthcam.xacro"/>
-    <xacro:VLP-16 parent="mount" name="velodyne" topic="/velodyne_points" hz="10" samples="440" gpu="${gpu}">
-        <origin xyz="0 0.195 0" rpy="-1.570796 -1.570796 0" />
+    <xacro:VLP-16 parent="base_link" name="velodyne" topic="/velodyne_points" hz="10" samples="440" gpu="${gpu}">
+        <origin xyz="0 -0.33 0.62" rpy="0 0 -1.5708" />
     </xacro:VLP-16>
-    <xacro:realsense_d435 sensor_name="d435" parent_link="mount" rate="10">
-        <origin xyz="0 0.1 0.28" rpy="0 -1.570796 -1.570796" />
+    <xacro:realsense_d435 sensor_name="d435" parent_link="base_link" rate="10">
+        <origin xyz="0 -0.38 0.58" rpy="0 0 -1.570796" />
     </xacro:realsense_d435>
     <gazebo>

Commit message: simulate 2D LiDAR

File: dependencies/catamaran/urdf/catamaran.urdf (robot description, URDF)
Before this commit: robot catamaran, 5 links, 4 joints
Links:
- added link laser_frame, mass 0; collision cylinder length=0.04 radius=0.05; visual cylinder length=0.04 radius=0.05
Joints:
- added joint laser_joint: type fixed, parent base_link, child laser_frame, origin xyz=0 -0.33 0.62 rpy=0 0 -1.570796

Commit message: added obstacles and 2D LiDAR simulation

File: dependencies/catamaran/urdf/catamaran.urdf (robot description, URDF)
Before this commit: robot catamaran, 6 links, 5 joints
Links:
- added link camera_link, mass 0
Joints:
- added joint base_to_camera: type fixed, parent base_link, child camera_link, origin xyz=0 0 3 rpy=0 0 0

File: triton/urdf/catamaran_full.urdf.xacro (robot description, xacro)
@@ -6,7 +6,7 @@
     <xacro:include filename="$(find velodyne_description)/urdf/VLP-16.urdf.xacro"/>
     <xacro:include filename="$(find realsense_ros_gazebo)/xacro/depthcam.xacro"/>
-    <xacro:VLP-16 parent="base_link" name="velodyne" topic="/velodyne_points" hz="10" samples="440" gpu="${gpu}">
+    <!-- <xacro:VLP-16 parent="base_link" name="velodyne" topic="/velodyne_points" hz="10" samples="440" gpu="${gpu}">
         <origin xyz="0 -0.33 0.62" rpy="0 0 -1.5708" />
-    </xacro:VLP-16>
+    </xacro:VLP-16> -->
     <xacro:realsense_d435 sensor_name="d435" parent_link="base_link" rate="10">
         <origin xyz="0 -0.38 0.58" rpy="0 0 -1.570796" />

Commit message: add hector mapping

File: dependencies/catamaran/urdf/catamaran.urdf (robot description, URDF)
Before this commit: robot catamaran, 7 links, 6 joints
Links:
- link base_link: geometry visual mesh filename=package://catamaran/meshes/base_link.STL

Commit message: mass overhaul to simulation

File: dependencies/catamaran/urdf/catamaran.urdf (robot description, URDF)
Before this commit: robot catamaran, 7 links, 6 joints
Links:
- removed link camera_link
- removed link laser_frame
- removed link waterwheel
- added link conveyor; collision mesh filename=package://catamaran/meshes/conveyor.STL; visual mesh filename=package://catamaran/meshes/conveyor.STL
- link base_link: mass 682.95 -> 65; geometry collision mesh filename=package://catamaran/meshes/base_link.STL; visual mesh filename=package://catamaran/meshes/base_link.STL
- link l_thruster: mass 4.9984 -> None
- link r_thruster: mass 0 -> None
Joints:
- removed joint base_to_camera
- removed joint base_to_l_thruster
- removed joint base_to_waterwheel
- removed joint laser_joint
- added joint base_to_conveyor: type fixed, parent base_link, child conveyor, origin xyz=0 -0.68537 0.44462 rpy=1.5708 0 0, axis 0 0 0
- added joint base_to_l_thrruster: type fixed, parent base_link, child l_thruster, origin xyz=0.55834 0.43963 -0.45538 rpy=1.5708 0 3.1416, axis 0 0 0
